Commit message: lidar_cam_simulation

File: urdf/bcr_bot.xacro (robot description, xacro)
@@ -27,5 +27,5 @@
     <xacro:arg name="wheel_odom_topic" default="odom"/>
     <xacro:arg name="camera_enabled" default="false"/>
-    <xacro:arg name="two_d_lidar_enabled" default="false"/>
+    <xacro:arg name="lidar_enabled" default="false"/>
     <xacro:arg name="publish_wheel_odom_tf" default="true"/>
     <xacro:arg name="conveyor_enabled" default="false"/>
@@ -218,16 +218,18 @@
     </xacro:if>
     <!-- ............................. LiDAR........................................ -->
-    <xacro:if value="$(arg camera_enabled)">
-        <link name="laser_livox">
-            <collision>
-                <origin xyz="0 0 0" rpy="0 0 0" />
-                <geometry>
-                    <box size="0.1 0.1 0.1"/>
-                </geometry>
-            </collision>
-            <visual>
-                <origin xyz="0 0 0" rpy="0 0 0" />
-                <geometry>
-                    <box size="0.1 0.1 0.1"/>
+    <xacro:if value="$(arg lidar_enabled)">
+        <link name="livox">
+            <collision>
+                <origin xyz="0 0 0" rpy="0 0 0" />
+                <geometry>
+                   <mesh filename="package://livox_laser_simulation/meshes/livox_mid40.dae">
+                   </mesh>
+                </geometry>
+            </collision>
+            <visual>
+                <origin xyz="0 0 0" rpy="0 0 0" />
+                <geometry>
+                    <mesh filename="package://livox_laser_simulation/meshes/livox_mid40.dae">
+          	</mesh>
                 </geometry>
                 <material name="black"/>
@@ -235,9 +237,9 @@
         </link>
         <joint name="laser_livox_joint" type="fixed">
-            <parent link="base_link"/>
-            <child link="laser_livox"/>
-            <origin xyz="0 0 0.2" rpy="0 0 0" />
-        </joint>
-        <gazebo reference="laser_livox"/>
+            <origin xyz="0 0 0.2" rpy="0 0 0"/>
+            <parent link="base_link"/>
+            <child link="livox"/>
+        </joint>
+        <gazebo reference="livox"/>
     </xacro:if>
     <!-- ............................. ROOF ........................................ -->

File: urdf/gazebo.xacro (robot description, xacro)
@@ -56,5 +56,5 @@
             <sensor type="camera" name="fisheye_camera">
                 <always_on>true</always_on>
-                <update_rate>30.0</update_rate>
+                <update_rate>20.0</update_rate>
                 <visualize>1</visualize>
                 <camera>
@@ -89,5 +89,5 @@
                     <cameraName>fisheye_camera</cameraName>
                     <alwaysOn>true</alwaysOn>
-                    <updateRateHZ>30.0</updateRateHZ>
+                    <updateRateHZ>20.0</updateRateHZ>
                     <imageTopicName>image_raw</imageTopicName>
                     <cameraInfoTopicName>camera_info</cameraInfoTopicName>
@@ -112,5 +112,5 @@
             <sensor type="camera" name="fisheye_camera2">
                 <always_on>true</always_on>
-                <update_rate>30.0</update_rate>
+                <update_rate>20.0</update_rate>
                 <visualize>1</visualize>
                 <camera>
@@ -145,5 +145,5 @@
                     <cameraName>fisheye_camera2</cameraName>
                     <alwaysOn>true</alwaysOn>
-                    <updateRateHZ>30.0</updateRateHZ>
+                    <updateRateHZ>20.0</updateRateHZ>
                     <imageTopicName>image_raw</imageTopicName>
                     <cameraInfoTopicName>camera_info</cameraInfoTopicName>
@@ -168,5 +168,5 @@
             <sensor type="camera" name="fisheye_camera3">
                 <always_on>true</always_on>
-                <update_rate>30.0</update_rate>
+                <update_rate>20.0</update_rate>
                 <visualize>1</visualize>
                 <camera>
@@ -201,5 +201,5 @@
                     <cameraName>fisheye_camera3</cameraName>
                     <alwaysOn>true</alwaysOn>
-                    <updateRateHZ>30.0</updateRateHZ>
+                    <updateRateHZ>20.0</updateRateHZ>
                     <imageTopicName>image_raw</imageTopicName>
                     <cameraInfoTopicName>camera_info</cameraInfoTopicName>
@@ -224,5 +224,5 @@
             <sensor type="camera" name="fisheye_camera4">
                 <always_on>true</always_on>
-                <update_rate>30.0</update_rate>
+                <update_rate>20.0</update_rate>
                 <visualize>1</visualize>
                 <camera>
@@ -257,5 +257,5 @@
                     <cameraName>fisheye_camera4</cameraName>
                     <alwaysOn>true</alwaysOn>
-                    <updateRateHZ>30.0</updateRateHZ>
+                    <updateRateHZ>20.0</updateRateHZ>
                     <imageTopicName>image_raw</imageTopicName>
                     <cameraInfoTopicName>camera_info</cameraInfoTopicName>
@@ -276,6 +276,6 @@
         </gazebo>
     </xacro:if>
-    <xacro:if value="$(arg camera_enabled)">
-        <gazebo reference="laser_livox">
+    <xacro:if value="$(arg lidar_enabled)">
+        <gazebo reference="livox">
             <sensor type="ray" name="laser_livox">
                 <pose>0 0 0 0 0 0</pose>
@@ -292,5 +292,5 @@
                         </horizontal>
                         <vertical>
-                        <samples>50</samples>
+                        <samples>360</samples>
                         <resolution>1</resolution>
                         <min_angle>${-vertical_fov/360*3.14159}</min_angle>
@@ -310,8 +310,8 @@
                     </ray>
                     <visualize>true</visualize>
-                    <samples>10000</samples>
+                    <samples>24000</samples>
                     <downsample>1</downsample>
-                    <csv_file_name>$(find bcr_bot)/meshes/livox/scan_mode/mid360.csv</csv_file_name>
-		  <ros_topic>scan</ros_topic>
+                    <csv_file_name>package://livox_laser_simulation/scan_mode/mid360.csv</csv_file_name>
+		  <ros_topic>$(arg robot_namespace)/livox/lidar</ros_topic>
                 </plugin>
             </sensor>
